Commit message: 添加z1和go1，修改了配置文件和控制器cpp

File: qm_description/urdf/qudraputed/robot.xacro (robot description, xacro)
@@ -1,5 +1,5 @@
 <?xml version="1.0"?>
 <robot xmlns:xacro="http://www.ros.org/wiki/xacro" name="robot">
-    <xacro:arg name="robot_type" default="aliengo"/>
+    <xacro:arg name="robot_type" default="go1"/>
     <xacro:include filename="$(find qm_description)/urdf/qudraputed/common/materials.xacro"/>
     <xacro:include filename="$(find qm_description)/urdf/qudraputed/common/leg.xacro"/>

File: qm_description/urdf/qudraputed_manipulator/robot.urdf (robot description, URDF)
Before this commit: robot qm, 27 links, 26 joints
Links:
- removed link arm_base_link
- removed link j2n6s300_end_effector
- removed link j2n6s300_link_1
- removed link j2n6s300_link_2
- removed link j2n6s300_link_3
- removed link j2n6s300_link_4
- removed link j2n6s300_link_5
- removed link j2n6s300_link_6
- removed link j2n6s300_link_base
- added link gripperMover, mass 0.27621302; collision mesh filename=package://qm_description/meshes/manipulator/z1_GripperMover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 scale=1 1 1; visual mesh filename=package://qm_description/meshes/manipulator/z1_GripperMover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 scale=1 1 1
- added link gripperStator, mass 0.52603655; collision mesh filename=package://qm_description/meshes/manipulator/z1_GripperStato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 scale=1 1 1; visual mesh filename=package://qm_description/meshes/manipulator/z1_GripperStato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 scale=1 1 1
- added link z1_end_effector, mass 0.0; collision sphere radius=0.01; visual sphere radius=0.01
- added link z1_link_0, mass 0.47247481; collision cylinder length=0.051 radius=0.0325; visual mesh filename=package://qm_description/meshes/manipulator/z1_Link00.stl scale=1 1 1
- added link z1_link_1, mass 0.67332551; collision cylinder length=0.102 radius=0.0325; visual mesh filename=package://qm_description/meshes/manipulator/z1_Link01.stl scale=1 1 1
- added link z1_link_2, mass 1.19132258; collision cylinder length=0.051 radius=0.0325; collision cylinder length=0.102 radius=0.0325
- added link z1_link_3, mass 0.83940874; collision cylinder length=0.059 radius=0.0325; collision cylinder length=0.116 radius=0.02
- added link z1_link_4, mass 0.56404563; collision cylinder length=0.067 radius=0.0325; visual mesh filename=package://qm_description/meshes/manipulator/z1_Link04.stl scale=1 1 1
- added link z1_link_5, mass 0.38938492; visual mesh filename=package://qm_description/meshes/manipulator/z1_Link05.stl scale=1 1 1
- added link z1_link_6, mass 0.28875807; collision cylinder length=0.051 radius=0.0325; visual mesh filename=package://qm_description/meshes/manipulator/z1_Link06.stl scale=1 1 1
- link LF_FOOT: geometry collision sphere radius=0.02; visual sphere radius=0.01
- link LF_calf: mass 0.207 -> 0.135862; geometry collision box size=0.213 0.016 0.016; visual mesh filename=package://qm_description/meshes/qudraputed/go1/calf.dae scale=1 1 1
- link LF_hip: mass 1.993 -> 0.591; geometry collision cylinder length=0.04 radius=0.046; visual mesh filename=package://qm_description/meshes/qudraputed/go1/hip.dae scale=1 1 1
- link LF_thigh: mass 0.639 -> 0.92; geometry collision box size=0.213 0.0245 0.034; collision cylinder length=0.032 radius=0.041
- link LH_FOOT: geometry collision sphere radius=0.02; visual sphere radius=0.01
- link LH_calf: mass 0.207 -> 0.135862; geometry collision box size=0.213 0.016 0.016; visual mesh filename=package://qm_description/meshes/qudraputed/go1/calf.dae scale=1 1 1
- link LH_hip: mass 1.993 -> 0.591; geometry collision cylinder length=0.04 radius=0.046; visual mesh filename=package://qm_description/meshes/qudraputed/go1/hip.dae scale=1 1 1
- link LH_thigh: mass 0.639 -> 0.92; geometry collision box size=0.213 0.0245 0.034; collision cylinder length=0.032 radius=0.041
- link RF_FOOT: geometry collision sphere radius=0.02; visual sphere radius=0.01
- link RF_calf: mass 0.207 -> 0.135862; geometry collision box size=0.213 0.016 0.016; visual mesh filename=package://qm_description/meshes/qudraputed/go1/calf.dae scale=1 1 1
- link RF_hip: mass 1.993 -> 0.591; geometry collision cylinder length=0.04 radius=0.046; visual mesh filename=package://qm_description/meshes/qudraputed/go1/hip.dae scale=1 1 1
- link RF_thigh: mass 0.639 -> 0.92; geometry collision box size=0.213 0.0245 0.034; collision cylinder length=0.032 radius=0.041
- link RH_FOOT: geometry collision sphere radius=0.02; visual sphere radius=0.01
- link RH_calf: mass 0.207 -> 0.135862; geometry collision box size=0.213 0.016 0.016; visual mesh filename=package://qm_description/meshes/qudraputed/go1/calf.dae scale=1 1 1
- link RH_hip: mass 1.993 -> 0.591; geometry collision cylinder length=0.04 radius=0.046; visual mesh filename=package://qm_description/meshes/qudraputed/go1/hip.dae scale=1 1 1
- link RH_thigh: mass 0.639 -> 0.92; geometry collision box size=0.213 0.0245 0.034; collision cylinder length=0.032 radius=0.041
- link base: mass 11.041 -> 5.204; geometry collision box size=0.3762 0.0935 0.114; visual mesh filename=package://qm_description/meshes/qudraputed/go1/trunk.dae scale=1 1 1
Joints:
- removed joint j2n6s300_joint_1
- removed joint j2n6s300_joint_2
- removed joint j2n6s300_joint_3
- removed joint j2n6s300_joint_4
- removed joint j2n6s300_joint_5
- removed joint j2n6s300_joint_6
- removed joint j2n6s300_joint_base
- removed joint j2n6s300_joint_end_effector
- added joint gripperStator: type fixed, parent z1_link_6, child gripperStator, origin xyz=0.051 0.0 0.0 rpy=0 0 0
- added joint z1_joint_1: type revolute, parent z1_link_0, child z1_link_1, origin xyz=0 0 0.0585 rpy=0 0 0, axis 0 0 1, limit lower=-2.6179938779914944 upper=2.6179938779914944 effort=30.0 velocity=3.1415
- added joint z1_joint_2: type revolute, parent z1_link_1, child z1_link_2, origin xyz=0 0 0.045 rpy=0 0 0, axis 0 1 0, limit lower=0.0 upper=2.9670597283903604 effort=60.0 velocity=3.1415
- added joint z1_joint_3: type revolute, parent z1_link_2, child z1_link_3, origin xyz=-0.35 0 0 rpy=0 0 0, axis 0 1 0, limit lower=-2.8797932657906435 upper=0.0 effort=30.0 velocity=3.1415
- added joint z1_joint_4: type revolute, parent z1_link_3, child z1_link_4, origin xyz=0.218 0 0.057 rpy=0 0 0, axis 0 1 0, limit lower=-1.5184364492350666 upper=1.5184364492350666 effort=30.0 velocity=3.1415
- added joint z1_joint_5: type revolute, parent z1_link_4, child z1_link_5, origin xyz=0.07 0.0 0.0 rpy=0 0 0, axis 0 0 1, limit lower=-1.3439035240356338 upper=1.3439035240356338 effort=30.0 velocity=3.1415
- added joint z1_joint_6: type revolute, parent z1_link_5, child z1_link_6, origin xyz=0.0492 0.0 0.0 rpy=0 0 0, axis 1 0 0, limit lower=-2.792526803190927 upper=2.792526803190927 effort=30.0 velocity=3.1415
- added joint z1_joint_Gripper: type fixed, parent gripperStator, child gripperMover, origin xyz=0.049 0.0 0 rpy=0 0 0, axis 0 1 0, limit lower=-1.5707963267948966 upper=0.0 effort=30.0 velocity=3.1415
- added joint z1_joint_end_effector: type fixed, parent gripperStator, child z1_end_effector, origin xyz=0.135 0 0 rpy=0 0 0
- joint LF_HAA: limit lower=-1.2217304763960306 upper=1.2217304763960306 effort=35.278 velocity=20 -> lower=-0.863 upper=0.863 effort=23.7 velocity=30.1; origin xyz=0.2407 0.051 0 rpy=0 0 0 -> xyz=0.1881 0.04675 0 rpy=0 0 0
- joint LF_HFE: limit lower=-1e+22 upper=1e+22 effort=35.278 velocity=20 -> lower=-0.686 upper=4.501 effort=23.7 velocity=30.1; origin xyz=0 0.0868 0 rpy=0 0 0 -> xyz=0 0.08 0 rpy=0 0 0
- joint LF_KFE: limit lower=-2.775073510670984 upper=-0.6457718232379019 effort=44.4 velocity=15.89 -> lower=-2.818 upper=-0.888 effort=35.55 velocity=20.06; origin xyz=0 0 -0.25 rpy=0 0 0 -> xyz=0 0 -0.213 rpy=0 0 0
- joint LF_foot_fixed: origin xyz=0 0 -0.25 rpy=0 0 0 -> xyz=0 0 -0.213 rpy=0 0 0
- joint LH_HAA: limit lower=-1.2217304763960306 upper=1.2217304763960306 effort=35.278 velocity=20 -> lower=-0.863 upper=0.863 effort=23.7 velocity=30.1; origin xyz=-0.2407 0.051 0 rpy=0 0 0 -> xyz=-0.1881 0.04675 0 rpy=0 0 0
- joint LH_HFE: limit lower=-1e+22 upper=1e+22 effort=35.278 velocity=20 -> lower=-0.686 upper=4.501 effort=23.7 velocity=30.1; origin xyz=0 0.0868 0 rpy=0 0 0 -> xyz=0 0.08 0 rpy=0 0 0
- joint LH_KFE: limit lower=-2.775073510670984 upper=-0.6457718232379019 effort=44.4 velocity=15.89 -> lower=-2.818 upper=-0.888 effort=35.55 velocity=20.06; origin xyz=0 0 -0.25 rpy=0 0 0 -> xyz=0 0 -0.213 rpy=0 0 0
- joint LH_foot_fixed: origin xyz=0 0 -0.25 rpy=0 0 0 -> xyz=0 0 -0.213 rpy=0 0 0
- joint RF_HAA: limit lower=-1.2217304763960306 upper=1.2217304763960306 effort=35.278 velocity=20 -> lower=-0.863 upper=0.863 effort=23.7 velocity=30.1; origin xyz=0.2407 -0.051 0 rpy=0 0 0 -> xyz=0.1881 -0.04675 0 rpy=0 0 0
- joint RF_HFE: limit lower=-1e+22 upper=1e+22 effort=35.278 velocity=20 -> lower=-0.686 upper=4.501 effort=23.7 velocity=30.1; origin xyz=0 -0.0868 0 rpy=0 0 0 -> xyz=0 -0.08 0 rpy=0 0 0
- joint RF_KFE: limit lower=-2.775073510670984 upper=-0.6457718232379019 effort=44.4 velocity=15.89 -> lower=-2.818 upper=-0.888 effort=35.55 velocity=20.06; origin xyz=0 0 -0.25 rpy=0 0 0 -> xyz=0 0 -0.213 rpy=0 0 0
- joint RF_foot_fixed: origin xyz=0 0 -0.25 rpy=0 0 0 -> xyz=0 0 -0.213 rpy=0 0 0
- joint RH_HAA: limit lower=-1.2217304763960306 upper=1.2217304763960306 effort=35.278 velocity=20 -> lower=-0.863 upper=0.863 effort=23.7 velocity=30.1; origin xyz=-0.2407 -0.051 0 rpy=0 0 0 -> xyz=-0.1881 -0.04675 0 rpy=0 0 0
- joint RH_HFE: limit lower=-1e+22 upper=1e+22 effort=35.278 velocity=20 -> lower=-0.686 upper=4.501 effort=23.7 velocity=30.1; origin xyz=0 -0.0868 0 rpy=0 0 0 -> xyz=0 -0.08 0 rpy=0 0 0
- joint RH_KFE: limit lower=-2.775073510670984 upper=-0.6457718232379019 effort=44.4 velocity=15.89 -> lower=-2.818 upper=-0.888 effort=35.55 velocity=20.06; origin xyz=0 0 -0.25 rpy=0 0 0 -> xyz=0 0 -0.213 rpy=0 0 0
- joint RH_foot_fixed: origin xyz=0 0 -0.25 rpy=0 0 0 -> xyz=0 0 -0.213 rpy=0 0 0
- joint manipulator_joint: child arm_base_link -> z1_link_0; origin xyz=0.0 0.0 0.01 rpy=0.0 0.0 0.0 -> xyz=0 0 0 rpy=0 0 0
