Commit message: 添加z1和go1，修改了配置文件和控制器cpp

File: qm_description/urdf/qudraputed_manipulator/robot_mpc.xacro (robot description, xacro)
@@ -2,15 +2,386 @@
 <robot xmlns:xacro="http://www.ros.org/wiki/xacro" name="qm">
     <!-- qudraputed -->
-    <xacro:arg name="robot_type" default="aliengo"/>
+    <xacro:arg name="robot_type" default="go1"/>
     <xacro:include filename="$(find qm_description)/urdf/qudraputed/robot.xacro" />
     <!-- manipulatior -->
-    <xacro:include filename="$(find qm_description)/urdf/manipulator/j2n6s300fix.xacro"/>
-    <link name="arm_base_link" />
+    <xacro:include filename="$(find qm_description)/urdf/manipulator/const.xacro"/>
+    <xacro:include filename="$(find qm_description)/urdf/manipulator/transmission.xacro"/>
     <joint name="manipulator_joint" type="fixed">
-        <parent link= "base" />
-        <child link = "arm_base_link" />
-        <origin xyz="0.0 0.0 0.01" rpy="0.0 0.0 0.0" />
-    </joint>
-    <xacro:j2n6s300  base_parent="arm_base_link"/>
+        <origin rpy="0 0 0" xyz="0 0 0"/>
+        <parent link="base"/>
+        <child link="z1_link_0"/>
+    </joint>
+    <xacro:arg name="UnitreeGripper" default="true"/>
+    <link name="z1_link_0">
+        <visual>
+            <origin rpy="0 0 0" xyz="0 0 0.057"/>
+            <geometry>
+                <mesh filename="package://qm_description/meshes/manipulator/z1_Link00.stl" scale="1 1 1"/>
+            </geometry>
+            <material name="silver"/>
+        </visual>
+        <collision>
+            <geometry>
+                <cylinder length="${motor_height}" radius="${motor_diameter}"/>
+            </geometry>
+            <origin rpy="0 0 0" xyz="0 0 ${motor_height/2.0}"/>
+        </collision>
+        <inertial>
+            <origin rpy="0 0 0" xyz="${L00_ComX} ${L00_ComY} ${L00_ComZ}"/>
+            <mass value="${L00_Mass}"/>
+            <inertia
+                ixx="${L00_Ixx}" ixy="${L00_Ixy}" ixz="${L00_Ixz}"
+                iyy="${L00_Iyy}" iyz="${L00_Iyz}"
+                izz="${L00_Izz}"/>
+        </inertial>
+    </link>
+   <joint name="z1_joint_1" type="revolute">
+        <origin rpy="0 0 0" xyz="0 0 0.0585"/>
+        <parent link="z1_link_0"/>
+        <child link="z1_link_1"/>
+        <axis xyz="0 0 1"/>
+        <dynamics damping="${jointDamping}" friction="${jointFriction}"/>
+        <limit effort="${torqueMax}" velocity="${velocityMax}" lower="${joint1_PositionMin}" upper="${joint1_PositionMax}"/>
+    </joint>
+    <xacro:motorTransmission name="1"/>
+    <gazebo>
+        <plugin filename="libgazebo_ros_ft_sensor.so" name="ft_sensor">
+        <updateRate>30.0</updateRate>
+        <topicName>z1_joint_1_ft_sensor_topic</topicName>
+        <jointName>z1_joint_1</jointName>
+        </plugin>
+    </gazebo>
+    <link name="z1_link_1">
+        <visual>
+            <origin rpy="0 0 0" xyz="0 0 0"/>
+            <geometry>
+                 <mesh filename="package://qm_description/meshes/manipulator/z1_Link01.stl" scale="1 1 1"/>
+            </geometry>
+            <material name="silver"/>
+        </visual>
+        <collision>
+            <geometry>
+                <cylinder length="${2*motor_height}" radius="${motor_diameter}"/>
+            </geometry>
+            <origin rpy="0 0 0" xyz="0 0 0"/>
+        </collision>
+        <inertial>
+            <origin rpy="0 0 0" xyz="${L01_ComX} ${L01_ComY} ${L01_ComZ}"/>
+            <mass value="${L01_Mass}"/>
+            <inertia
+                ixx="${L01_Ixx}" ixy="${L01_Ixy}" ixz="${L01_Ixz}"
+                iyy="${L01_Iyy}" iyz="${L01_Iyz}"
+                izz="${L01_Izz}"/>
+        </inertial>
+    </link>
+    <joint name="z1_joint_2" type="revolute">
+        <origin rpy="0 0 0" xyz="0 0 0.045"/>
+        <parent link="z1_link_1"/>
+        <child link="z1_link_2"/>
+        <axis xyz="0 1 0"/>
+        <dynamics damping="${2*jointDamping}" friction="${2*jointFriction}"/>
+        <limit effort="${2*torqueMax}" velocity="${velocityMax}" lower="${joint2_PositionMin}" upper="${joint2_PositionMax}"/>
+    </joint>
+    <xacro:motorTransmission name="2"/>
+    <gazebo>
+        <plugin filename="libgazebo_ros_ft_sensor.so" name="ft_sensor">
+        <updateRate>30.0</updateRate>
+        <topicName>z1_joint_2_ft_sensor_topic</topicName>
+        <jointName>z1_joint_2</jointName>
+        </plugin>
+    </gazebo>
+    <link name="z1_link_2">
+        <visual>
+            <origin rpy="0 0 0" xyz="0 0 0"/>
+            <geometry>
+                <mesh filename="package://qm_description/meshes/manipulator/z1_Link02.stl" scale="1 1 1"/>
+            </geometry>
+            <material name="silver"/>
+        </visual>
+        <collision>
+            <geometry>
+                <cylinder length="${2.0*motor_height}" radius="${motor_diameter}"/>
+            </geometry>
+            <origin rpy="${PI/2.0} 0 0" xyz="0 0 0"/>
+        </collision>
+        <collision>
+            <geometry>
+                <cylinder length="${arm1_height}" radius="${arm1_diameter}"/>
+            </geometry>
+            <origin rpy="0 ${PI/2.0} 0" xyz="${-0.045-arm1_height/2.0} 0 0"/>
+        </collision>
+        <collision>
+            <geometry>
+                <cylinder length="${motor_height}" radius="${motor_diameter}"/>
+            </geometry>
+            <origin rpy="${PI/2.0} 0 0" xyz="-0.35 0 0"/>
+        </collision>
+        <inertial>
+            <origin rpy="0 0 0" xyz="${L02_ComX} ${L02_ComY} ${L02_ComZ}"/>
+            <mass value="${L02_Mass}"/>
+            <inertia
+                ixx="${L02_Ixx}" ixy="${L02_Ixy}" ixz="${L02_Ixz}"
+                iyy="${L02_Iyy}" iyz="${L02_Iyz}"
+                izz="${L02_Izz}"/>
+        </inertial>
+    </link>
+    <joint name="z1_joint_3" type="revolute">
+        <origin rpy="0 0 0" xyz="-0.35 0 0"/>
+        <parent link="z1_link_2"/>
+        <child link="z1_link_3"/>
+        <axis xyz="0 1 0"/>
+        <dynamics damping="${jointDamping}" friction="${jointFriction}"/>
+        <limit effort="${torqueMax}" velocity="${velocityMax}" lower="${joint3_PositionMin}" upper="${joint3_PositionMax}"/>
+    </joint>
+    <xacro:motorTransmission name="3"/>
+    <gazebo>
+        <plugin filename="libgazebo_ros_ft_sensor.so" name="ft_sensor">
+        <updateRate>30.0</updateRate>
+        <topicName>z1_joint_3_ft_sensor_topic</topicName>
+        <jointName>z1_joint_3</jointName>
+        </plugin>
+    </gazebo>
+    <link name="z1_link_3">
+        <visual>
+            <origin rpy="0 0 0" xyz="0 0 0"/>
+            <geometry>
+                <mesh filename="package://qm_description/meshes/manipulator/z1_Link03.stl" scale="1 1 1"/>
+            </geometry>
+            <material name="silver"/>
+        </visual>
+        <collision>
+            <geometry>
+                <cylinder length="${arm2_height-0.01}" radius="${arm2_diameter}"/>
+            </geometry>
+            <origin rpy="0 ${PI/2.0} 0" xyz="${0.065+arm2_height/2.0} 0 0.055"/>
+        </collision>
+        <collision>
+            <geometry>
+                <cylinder length="0.059" radius="${motor_diameter}"/>
+            </geometry>
+            <origin rpy="0 ${PI/2.0} ${PI/2.0}" xyz="${0.065+0.185-0.059/2.0} 0 0.055"/>
+        </collision>
+        <inertial>
+            <origin rpy="0 0 0" xyz="${L03_ComX} ${L03_ComY} ${L03_ComZ}"/>
+            <mass value="${L03_Mass}"/>
+            <inertia
+                ixx="${L03_Ixx}" ixy="${L03_Ixy}" ixz="${L03_Ixz}"
+                iyy="${L03_Iyy}" iyz="${L03_Iyz}"
+                izz="${L03_Izz}"/>
+        </inertial>
+    </link>
+    <joint name="z1_joint_4" type="revolute">
+        <origin rpy="0 0 0" xyz="0.218 0 0.057"/>
+        <parent link="z1_link_3"/>
+        <child link="z1_link_4"/>
+        <axis xyz="0 1 0"/>
+        <dynamics damping="${jointDamping}" friction="${jointFriction}"/>
+        <limit effort="${torqueMax}" velocity="${velocityMax}" lower="${joint4_PositionMin}" upper="${joint4_PositionMax}"/>
+    </joint>
+    <xacro:motorTransmission name="4"/>
+    <gazebo>
+        <plugin filename="libgazebo_ros_ft_sensor.so" name="ft_sensor">
+        <updateRate>30.0</updateRate>
+        <topicName>z1_joint_4_ft_sensor_topic</topicName>
+        <jointName>z1_joint_4</jointName>
+        </plugin>
+    </gazebo>
+    <link name="z1_link_4">
+        <visual>
+            <origin rpy="0 0 0" xyz="0 0 0"/>
+            <geometry>
+                 <mesh filename="package://qm_description/meshes/manipulator/z1_Link04.stl" scale="1 1 1"/>
+            </geometry>
+            <material name="silver"/>
+        </visual>
+        <collision>
+            <geometry>
+                <cylinder length="${motor_height + 2*0.008}" radius="${motor_diameter}"/>
+            </geometry>
+            <origin rpy="0 0 0" xyz="0.072 0 0"/>
+        </collision>
+        <inertial>
+            <origin rpy="0 0 0" xyz="${L04_ComX} ${L04_ComY} ${L04_ComZ}"/>
+            <mass value="${L04_Mass}"/>
+            <inertia
+                ixx="${L04_Ixx}" ixy="${L04_Ixy}" ixz="${L04_Ixz}"
+                iyy="${L04_Iyy}" iyz="${L04_Iyz}"
+                izz="${L04_Izz}"/>
+        </inertial>
+    </link>
+    <joint name="z1_joint_5" type="revolute">
+        <origin rpy="0 0 0" xyz="0.07 0.0 0.0"/>
+        <parent link="z1_link_4"/>
+        <child link="z1_link_5"/>
+        <axis xyz="0 0 1"/>
+        <dynamics damping="${jointDamping}" friction="${jointFriction}"/>
+        <limit effort="${torqueMax}" velocity="${velocityMax}" lower="${joint5_PositionMin}" upper="${joint5_PositionMax}"/>
+    </joint>
+    <xacro:motorTransmission name="5"/>
+    <gazebo>
+        <plugin filename="libgazebo_ros_ft_sensor.so" name="ft_sensor">
+        <updateRate>30.0</updateRate>
+        <topicName>z1_joint_5_ft_sensor_topic</topicName>
+        <jointName>z1_joint_5</jointName>
+        </plugin>
+    </gazebo>
+    <link name="z1_link_5">
+        <visual>
+            <origin rpy="0 0 0" xyz="0 0 0"/>
+            <geometry>
+                <mesh filename="package://qm_description/meshes/manipulator/z1_Link05.stl" scale="1 1 1"/>
+            </geometry>
+            <material name="silver"/>
+        </visual>
+        <inertial>
+            <origin rpy="0 0 0" xyz="${L05_ComX} ${L05_ComY} ${L05_ComZ}"/>
+            <mass value="${L05_Mass}"/>
+            <inertia
+                ixx="${L05_Ixx}" ixy="${L05_Ixy}" ixz="${L05_Ixz}"
+                iyy="${L05_Iyy}" iyz="${L05_Iyz}"
+                izz="${L05_Izz}"/>
+        </inertial>
+    </link>
+    <joint name="z1_joint_6" type="revolute">
+        <origin rpy="0 0 0" xyz="0.0492 0.0 0.0"/>
+        <parent link="z1_link_5"/>
+        <child link="z1_link_6"/>
+        <axis xyz="1 0 0"/>
+        <dynamics damping="${jointDamping}" friction="${jointFriction}"/>
+        <limit effort="${torqueMax}" velocity="${velocityMax}" lower="${joint6_PositionMin}" upper="${joint6_PositionMax}"/>
+    </joint>
+    <xacro:motorTransmission name="6"/>
+    <gazebo>
+        <plugin filename="libgazebo_ros_ft_sensor.so" name="ft_sensor">
+        <updateRate>30.0</updateRate>
+        <topicName>z1_joint_6_ft_sensor_topic</topicName>
+        <jointName>z1_joint_6</jointName>
+        </plugin>
+    </gazebo>
+    <link name="z1_link_6">
+        <visual>
+            <origin rpy="0 0 0" xyz="0 0 0"/>
+            <geometry>
+                <mesh filename="package://qm_description/meshes/manipulator/z1_Link06.stl" scale="1 1 1"/>
+            </geometry>
+            <material name="silver"/>
+        </visual>
+        <collision>
+            <geometry>
+                <cylinder length="${motor_height}" radius="${motor_diameter}"/>
+            </geometry>
+            <origin rpy="0 ${PI/2.0} 0" xyz="${motor_height/2.0} 0 0"/>
+        </collision>
+        <inertial>
+            <origin rpy="0 0 0" xyz="${L06_ComX} ${L06_ComY} ${L06_ComZ}"/>
+            <mass value="${L06_Mass}"/>
+            <inertia
+                ixx="${L06_Ixx}" ixy="${L06_Ixy}" ixz="${L06_Ixz}"
+                iyy="${L06_Iyy}" iyz="${L06_Iyz}"
+                izz="${L06_Izz}"/>
+        </inertial>
+    </link>
+   <xacro:if value="$(arg UnitreeGripper)" >
+        <joint name="gripperStator" type="fixed">
+            <origin rpy="0 0 0" xyz="0.051 0.0 0.0"/>
+            <parent link="z1_link_6"/>
+            <child link="gripperStator"/>
+        </joint>
+        <link name="gripperStator">
+            <visual>
+                <geometry>
+                    <mesh filename="package://qm_description/meshes/manipulator/z1_GripperStator.stl" scale="1 1 1"/>
+                </geometry>
+                <material name="black"/>
+            </visual>
+            <collision>
+                <geometry>
+                    <mesh filename="package://qm_description/meshes/manipulator/z1_GripperStator.stl" scale="1 1 1"/>
+                </geometry>
+                <material name="green"/>
+            </collision>
+            <inertial>
+                <origin rpy="0 0 0" xyz="${GripperStator_ComX} ${GripperStator_ComY} ${GripperStator_ComZ}"/>
+                <mass value="${GripperStator_Mass}"/>
+                <inertia
+                    ixx="${GripperStator_Ixx}" ixy="${GripperStator_Ixy}" ixz="${GripperStator_Ixz}"
+                    iyy="${GripperStator_Iyy}" iyz="${GripperStator_Iyz}"
+                    izz="${GripperStator_Izz}"/>
+            </inertial>
+        </link>
+        <!-- TODO Change to revolute once controller is programmed -->
+        <joint name="z1_joint_Gripper" type="fixed">
+            <origin rpy="0 0 0" xyz="0.049 0.0 0"/>
+            <parent link="gripperStator"/>
+            <child link="gripperMover"/>
+            <axis xyz="0 1 0"/>
+            <dynamics damping="${jointDamping}" friction="${jointFriction}"/>
+            <limit effort="${torqueMax}" velocity="${velocityMax}" lower="${Gripper_PositionMin}" upper="${Gripper_PositionMax}"/>
+        </joint>
+<!--        <transmission name="z1_joint_Gripper_trans">-->
+<!--            <type>transmission_interface/SimpleTransmission</type>-->
+<!--            <joint name="z1_joint_Gripper">-->
+<!--                <hardwareInterface>hardware_interface/EffortJointInterface</hardwareInterface>-->
+<!--            </joint>-->
+<!--            <actuator name="z1_joint_Gripper_motor">-->
+<!--                <mechanicalReduction>1</mechanicalReduction>-->
+<!--            </actuator>-->
+<!--        </transmission>-->
+        <!-- <gazebo>
+            <plugin name="gripper_position_controller" filename="libgazebo_ros_control_select_joints.so">
+                <robotNamespace>/</robotNamespace>
+                <joints>z1_joint_Gripper</joints>
+            </plugin>
+        </gazebo> -->
+        <link name="gripperMover">
+            <visual>
+                <geometry>
+                    <mesh filename="package://qm_description/meshes/manipulator/z1_GripperMover.stl" scale="1 1 1"/>
+                </geometry>
+                <material name="black"/>
+            </visual>
+            <collision>
+                <geometry>
+                    <mesh filename="package://qm_description/meshes/manipulator/z1_GripperMover.stl" scale="1 1 1"/>
+                </geometry>
+                <material name="green"/>
+            </collision>
+            <inertial>
+                <origin rpy="0 0 0" xyz="${GripperMover_ComX} ${GripperMover_ComY} ${GripperMover_ComZ}"/>
+                <mass value="${GripperMover_Mass}"/>
+                <inertia
+                    ixx="${GripperMover_Ixx}" ixy="${GripperMover_Ixy}" ixz="${GripperMover_Ixz}"
+                    iyy="${GripperMover_Iyy}" iyz="${GripperMover_Iyz}"
+                    izz="${GripperMover_Izz}"/>
+            </inertial>
+        </link>
+        <link name="z1_end_effector">
+            <visual>
+                <geometry>
+                    <sphere radius="0.01"/>
+                </geometry>
+                <material name="red"/>
+            </visual>
+            <inertial>
+                <mass value="0.0"/>
+                <inertia ixx="0.0" ixy="0.0" ixz="0.0" iyy="0.0" iyz="0.0" izz="0.0"/>
+            </inertial>
+            <collision>
+                <geometry>
+                    <sphere radius="0.01"/>
+                </geometry>
+                <surface>
+                    <contact>
+                        <collide_bitmask>0</collide_bitmask>
+                    </contact>
+                </surface>
+            </collision>
+        </link>
+        <joint name="z1_joint_end_effector" type="fixed">
+            <origin xyz="0.135 0 0" rpy="0 0 0"/>
+            <parent link="gripperStator"/>
+            <child link="z1_end_effector"/>
+        </joint>
+    </xacro:if>
     <!-- ros_control plugin -->
     <gazebo>
